Commit message: Task 1.3.1.2: Remade URDF

File: urdf/robotaxi.urdf (robot description, URDF)
Before this commit: robot robotaxi, 13 links, 12 joints
Links:
- added link side_pane_1, mass 269.579902102743; collision mesh filename=package://project_legion/meshes/side_pane_1.STL; visual mesh filename=package://project_legion/meshes/side_pane_1.STL
- added link side_pane_2, mass 269.579902102743; collision mesh filename=package://project_legion/meshes/side_pane_2.STL; visual mesh filename=package://project_legion/meshes/side_pane_2.STL
- added link side_pane_3, mass 238.283902102743; collision mesh filename=package://project_legion/meshes/side_pane_3.STL; visual mesh filename=package://project_legion/meshes/side_pane_3.STL
- added link side_pane_4, mass 238.283902102743; collision mesh filename=package://project_legion/meshes/side_pane_4.STL; visual mesh filename=package://project_legion/meshes/side_pane_4.STL
- added link top, mass 1431.79274848221; collision mesh filename=package://project_legion/meshes/top.STL; visual mesh filename=package://project_legion/meshes/top.STL
- link back_left_wheel: mass 220.204654088326 -> 220.204654088327
- link body: mass 7062.99841256932 -> 4615.47805567614
Joints:
- added joint side_pane_1_joint: type fixed, parent body, child side_pane_1, origin xyz=0 0 0 rpy=0 0 0, axis 0 0 0
- added joint side_pane_2_joint: type fixed, parent body, child side_pane_2, origin xyz=0 0 0 rpy=0 0 0, axis 0 0 0
- added joint side_pane_3_joint: type fixed, parent body, child side_pane_3, origin xyz=0 0 0 rpy=0 0 0, axis 0 0 0
- added joint side_pane_4_joint: type fixed, parent body, child side_pane_4, origin xyz=2 0 1 rpy=-1.5708 0 -1.5708, axis 0 0 0
- added joint top_joint: type fixed, parent body, child top, origin xyz=0 0 0 rpy=0 0 0, axis 0 0 0
- joint back_left_wheel_joint: axis -0.10781 -0.99417 0 -> -0.107805398797207 -0.99417201529221 0
- joint back_right_wheel_joint: axis -0.054755 0.9985 0 -> -0.0547547589597665 0.998499832935018 0
- joint front_left_wheel_joint: axis -0.62337 -0.78192 0 -> -0.623373961813521 -0.781923847783731 0
- joint front_right_wheel_joint: axis 0.08222 0.99661 0 -> 0.0822198916962624 0.996614212927678 0

Commit message: Task 1.3.1.3: Remade URDF

File: urdf/robotaxi.urdf (robot description, URDF)
Before this commit: robot robotaxi, 18 links, 17 joints
Joints:
- joint side_pane_4_joint: origin xyz=2 0 1 rpy=-1.5708 0 -1.5708 -> xyz=2 0 1 rpy=-1.5707963267949 0 -1.5707963267949
