Commit message: Task 1.3.3: Updated URDF

File: urdf/robotaxi_old.urdf.xacro (robot description, xacro)
@@ -1,8 +1,8 @@
-<?xml version="1.0"?>
+<?xml version="1.0" ?>
 <!-- This URDF was automatically created by SolidWorks to URDF Exporter! Originally created by Stephen Brawner (brawner@gmail.com)
      Commit Version: 1.6.0-4-g7f85cfe  Build Version: 1.6.7995.38578
      For more information, please see http://wiki.ros.org/sw_urdf_exporter -->
 <robot
-  name="robotaxi">
+  name="robotaxi" xmlns:xacro="http://ros.org/wiki/xacro">
   <xacro:macro name="body_color">
   <visual>
@@ -69,5 +69,5 @@
     <inertial>
       <origin
-        xyz="-5.21780361656553E-05 -2.37407212439034E-05 0.604812969920948"
+        xyz="-5.21780361655602E-05 -2.37407212439023E-05 0.604812969920948"
         rpy="0 0 0" />
       <mass
@@ -75,9 +75,9 @@
       <inertia
         ixx="1863.24455406167"
-        ixy="0.0132219930650691"
-        ixz="-0.0745602857101254"
+        ixy="0.0132219930650718"
+        ixz="-0.0745602857100425"
         iyy="8715.44296968045"
-        iyz="-0.0273565484551131"
-        izz="9003.50747380203" />
+        iyz="-0.0273565484550983"
+        izz="9003.50747380204" />
     </inertial>
     <visual>
@@ -109,5 +109,5 @@
     <inertial>
       <origin
-        xyz="-0.00745692269118803 -0.090387884139878 0.106936663484027"
+        xyz="1.59254307730881 -0.770387884139879 0.306936663484025"
         rpy="0 0 0" />
       <mass
@@ -149,5 +149,5 @@
     type="revolute">
     <origin
-      xyz="1.6 -0.680000000000001 0.199999999999998"
+      xyz="0 0 0"
       rpy="0 0 0" />
     <parent
@@ -167,5 +167,5 @@
     <inertial>
       <origin
-        xyz="-6.45153368084017E-05 -0.000782011509483205 -1.11022302462516E-16"
+        xyz="1.57025410376083 -1.04055974237639 0.309999999999996"
         rpy="0 0 0" />
       <mass
@@ -174,7 +174,7 @@
         ixx="19.7127728680101"
         ixy="1.16262531983733"
-        ixz="5.60424286950757E-15"
+        ixz="5.70065896608079E-15"
         iyy="33.7094191498882"
-        iyz="5.89373897821999E-14"
+        iyz="5.93281734338829E-14"
         izz="19.6168571900673" />
     </inertial>
@@ -205,7 +205,7 @@
   <joint
     name="front_right_wheel_joint"
-    type="revolute">
-    <origin
-      xyz="-0.0296813809023602 -0.359777730866907 0.109999999999998"
+    type="continuous">
+    <origin
+      xyz="0 0 0"
       rpy="0 0 0" />
     <parent
@@ -225,5 +225,5 @@
     <inertial>
       <origin
-        xyz="0.0565368692558958 0.0709165541990985 0.106936664135948"
+        xyz="1.6565368692559 0.750916554199098 0.30693666413595"
         rpy="0 0 0" />
       <mass
@@ -265,5 +265,5 @@
     type="revolute">
     <origin
-      xyz="1.6 0.68 0.200000000000002"
+      xyz="0 0 0"
       rpy="0 0 0" />
     <parent
@@ -283,5 +283,5 @@
     <inertial>
       <origin
-        xyz="0.000489141742639143 0.000613550800876106 -5.55111512312578E-17"
+        xyz="1.82552714195732 0.962888059850802 0.310000000000004"
         rpy="0 0 0" />
       <mass
@@ -290,7 +290,7 @@
         ixx="25.1304300235974"
         ixy="6.91590337281265"
-        ixz="2.78048991352224E-14"
+        ixz="2.78109008982202E-14"
         iyy="28.2917619943008"
-        iyz="2.83576334348763E-14"
+        iyz="2.83392710451218E-14"
         izz="19.6168571900673" />
     </inertial>
@@ -321,7 +321,7 @@
   <joint
     name="front_left_wheel_joint"
-    type="revolute">
-    <origin
-      xyz="0.22503800021468 0.282274509049927 0.110000000000001"
+    type="continuous">
+    <origin
+      xyz="0 0 0"
       rpy="0 0 0" />
     <parent
@@ -341,5 +341,5 @@
     <inertial>
       <origin
-        xyz="0.0097773994104382 0.0901663896845278 0.106936663157124"
+        xyz="-1.59022260058956 0.770166389684527 0.306936663157127"
         rpy="0 0 0" />
       <mass
@@ -381,5 +381,5 @@
     type="revolute">
     <origin
-      xyz="-1.6 0.679999999999999 0.200000000000002"
+      xyz="0 0 0"
       rpy="0 0 0" />
     <parent
@@ -399,5 +399,5 @@
     <inertial>
       <origin
-        xyz="8.45914713538676E-05 0.000780095194589547 5.55111512312578E-17"
+        xyz="-1.56099765956285 1.03967619271508 0.310000000000004"
         rpy="0 0 0" />
       <mass
@@ -406,7 +406,7 @@
         ixx="19.7817557340667"
         ixy="1.52068003676715"
-        ixz="-1.4753654276074E-16"
+        ixz="-1.41066843422813E-16"
         iyy="33.6404362838315"
-        iyz="5.35549915294688E-14"
+        iyz="5.35623170831363E-14"
         izz="19.6168571900673" />
     </inertial>
@@ -437,7 +437,7 @@
   <joint
     name="back_left_wheel_joint"
-    type="revolute">
-    <origin
-      xyz="0.0389177489657917 0.358896097520487 0.110000000000001"
+    type="continuous">
+    <origin
+      xyz="0 0 0"
       rpy="0 0 0" />
     <parent
@@ -457,5 +457,5 @@
     <inertial>
       <origin
-        xyz="0.00496598832173212 -0.0905588974643843 0.106936665235941"
+        xyz="-1.59503401167827 -0.770558897464385 0.306936665235939"
         rpy="0 0 0" />
       <mass
@@ -497,5 +497,5 @@
     type="revolute">
     <origin
-      xyz="-1.6 -0.680000000000001 0.199999999999998"
+      xyz="0 0 0"
       rpy="0 0 0" />
     <parent
@@ -515,5 +515,5 @@
     <inertial>
       <origin
-        xyz="4.29643197439322E-05 -0.000783491095595057 1.66533453693773E-16"
+        xyz="-1.58019056769578 -1.04124193078514 0.309999999999997"
         rpy="0 0 0" />
       <mass
@@ -522,7 +522,7 @@
         ixx="19.6593954325899"
         ixy="-0.775721213261626"
-        ixz="-1.12194595756566E-15"
+        ixz="-1.12449279054662E-15"
         iyy="33.7627965853084"
-        iyz="5.12561448128763E-14"
+        iyz="5.12487286095604E-14"
         izz="19.6168571900673" />
     </inertial>
@@ -553,7 +553,7 @@
   <joint
     name="back_right_wheel_joint"
-    type="revolute">
-    <origin
-      xyz="0.0197664679844756 -0.360458439689542 0.109999999999999"
+    type="continuous">
+    <origin
+      xyz="0 0 0"
       rpy="0 0 0" />
     <parent
@@ -573,5 +573,5 @@
     <inertial>
       <origin
-        xyz="-0.0040420953035909 0.00404209530359112 -0.131846445933433"
+        xyz="2.10240622729717 -1.10240622729716 1.78815355406656"
         rpy="0 0 0" />
       <mass
@@ -579,8 +579,8 @@
       <inertia
         ixx="0.0642189157299355"
-        ixy="-0.000191353707477662"
-        ixz="0.00017449312202714"
+        ixy="-0.000191353707477661"
+        ixz="0.000174493122027139"
         iyy="0.0642189157299355"
-        iyz="-0.000174493122027057"
+        iyz="-0.000174493122027053"
         izz="0.0429541548113749" />
     </inertial>
@@ -613,5 +613,5 @@
     type="fixed">
     <origin
-      xyz="2.10644832260076 -1.10644832260075 1.92"
+      xyz="0 0 0"
       rpy="0 0 0" />
     <parent
@@ -626,5 +626,5 @@
     <inertial>
       <origin
-        xyz="-0.0040420953035909 -0.00404209530359023 -0.131846445933433"
+        xyz="2.10240622729716 1.10240622729716 1.78815355406657"
         rpy="0 0 0" />
       <mass
@@ -666,5 +666,5 @@
     type="fixed">
     <origin
-      xyz="2.10644832260075 1.10644832260076 1.92"
+      xyz="0 0 0"
       rpy="0 0 0" />
     <parent
@@ -679,5 +679,5 @@
     <inertial>
       <origin
-        xyz="0.00404209530359001 -0.00404209530359023 -0.131846445933433"
+        xyz="-2.10240622729717 1.10240622729715 1.78815355406657"
         rpy="0 0 0" />
       <mass
@@ -719,5 +719,5 @@
     type="fixed">
     <origin
-      xyz="-2.10644832260076 1.10644832260074 1.92"
+      xyz="0 0 0"
       rpy="0 0 0" />
     <parent
@@ -732,5 +732,5 @@
     <inertial>
       <origin
-        xyz="0.00404209530359001 0.0040420953035909 -0.131846445933433"
+        xyz="-2.10240622729716 -1.10240622729717 1.78815355406656"
         rpy="0 0 0" />
       <mass
@@ -772,5 +772,5 @@
     type="fixed">
     <origin
-      xyz="-2.10644832260075 -1.10644832260076 1.92"
+      xyz="0 0 0"
       rpy="0 0 0" />
     <parent
@@ -785,5 +785,5 @@
     <inertial>
       <origin
-        xyz="1.16326750898592E-16 -0.0600000000000008 0.225785335083629"
+        xyz="1.19387690613411E-15 0.939999999999996 1.22578533508363"
         rpy="0 0 0" />
       <mass
@@ -791,8 +791,8 @@
       <inertia
         ixx="29.0495518679719"
-        ixy="-1.20383938267796E-16"
-        ixz="2.77270150877661E-14"
+        ixy="-1.20383938267813E-16"
+        ixz="3.27421223583015E-14"
         iyy="417.804106229136"
-        iyz="9.90699315364669E-14"
+        iyz="9.89684859766926E-14"
         izz="389.401546126211" />
     </inertial>
@@ -825,5 +825,5 @@
     type="fixed">
     <origin
-      xyz="0 0.999999999999997 1"
+      xyz="0 0 0"
       rpy="0 0 0" />
     <parent
@@ -838,5 +838,5 @@
     <inertial>
       <origin
-        xyz="1.42066406747502E-16 -0.0600000000000011 0.225785335083629"
+        xyz="7.36854275917892E-17 -0.940000000000004 1.22578533508363"
         rpy="0 0 0" />
       <mass
@@ -844,8 +844,8 @@
       <inertia
         ixx="29.0495518679719"
-        ixy="-1.20383938267802E-16"
-        ixz="2.95831600997074E-14"
+        ixy="-1.20383938267801E-16"
+        ixz="2.9415137108934E-14"
         iyy="417.804106229136"
-        iyz="9.90076534888227E-14"
+        iyz="9.89935929190605E-14"
         izz="389.401546126211" />
     </inertial>
@@ -878,5 +878,5 @@
     type="fixed">
     <origin
-      xyz="0 -0.88 1"
+      xyz="0 0 0"
       rpy="0 0 0" />
     <parent
@@ -891,5 +891,5 @@
     <inertial>
       <origin
-        xyz="0.0600000000000001 -5.31535442847841E-16 0.16174583422535"
+        xyz="-1.94 -4.0299328481463E-15 1.16174583422535"
         rpy="0 0 0" />
       <mass
@@ -900,5 +900,5 @@
         ixz="1.67397202198221E-16"
         iyy="30.1909069158719"
-        iyz="-1.15365873460716E-13"
+        iyz="-1.1589443866755E-13"
         izz="61.6255164977819" />
     </inertial>
@@ -931,5 +931,5 @@
     type="fixed">
     <origin
-      xyz="-2 0 1"
+      xyz="0 0 0"
       rpy="0 0 0" />
     <parent
@@ -944,15 +944,15 @@
     <inertial>
       <origin
-        xyz="-0.0599999999999998 -6.46632113124857E-16 0.16174583422535"
+        xyz="8.11876186905901E-17 -0.16174583422535 -0.0599999999999998"
         rpy="0 0 0" />
       <mass
         value="238.283902102743" />
       <inertia
-        ixx="91.2445420486072"
-        ixy="-3.03407211392028E-16"
-        ixz="-4.15490215971411E-16"
-        iyy="30.1909069158719"
-        iyz="-1.23477209187437E-13"
-        izz="61.6255164977819" />
+        ixx="30.1909069158719"
+        ixy="-1.35061898246685E-14"
+        ixz="3.03407211392029E-16"
+        iyy="61.6255164977819"
+        iyz="4.1134269100746E-16"
+        izz="91.2445420486072" />
     </inertial>
     <visual>
@@ -985,5 +985,5 @@
     <origin
       xyz="2 0 1"
-      rpy="0 0 0" />
+      rpy="-1.5707963267949 0 -1.5707963267949" />
     <parent
       link="body" />
@@ -997,5 +997,5 @@
     <inertial>
       <origin
-        xyz="1.11795670913679E-15 -4.75570435698576E-17 -0.161525009353001"
+        xyz="1.579007960937E-15 -8.23001329418906E-15 2.058474990647"
         rpy="0 0 0" />
       <mass
@@ -1004,7 +1004,7 @@
         ixx="675.858793348103"
         ixy="-0.000168194562486687"
-        ixz="5.06178673563019E-13"
+        ixz="5.13110389472562E-13"
         iyy="2286.6645250204"
-        iyz="-1.99421702931628E-12"
+        iyz="-1.99695025936543E-12"
         izz="2900.47257026417" />
     </inertial>
@@ -1037,5 +1037,5 @@
     type="fixed">
     <origin
-      xyz="0 0 2.22"
+      xyz="0 0 0"
       rpy="0 0 0" />
     <parent
@@ -1046,5 +1046,5 @@
       xyz="0 0 0" />
   </joint>
-   <gazebo reference="body">
+  <gazebo reference="body">
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