Commit message: Task 1.4.1: Added Launch File to Spwan Robot

File: urdf/robotaxi.urdf.xacro (robot description, xacro)
@@ -3,20 +3,81 @@
      Commit Version: 1.6.0-4-g7f85cfe  Build Version: 1.6.7995.38578
      For more information, please see http://wiki.ros.org/sw_urdf_exporter -->
-<robot  name="robotaxi" xmlns:xacro="http://ros.org/wiki/xacro">
+<robot
+  name="robotaxi" xmlns:xacro="http://ros.org/wiki/xacro">
+  <xacro:macro name="body_color">
+  <visual>
+    <material>
+      <ambient>0.250980392156863 0.250980392156863 0.250980392156863 1</ambient>
+      <diffuse>0.250980392156863 0.250980392156863 0.250980392156863 1</diffuse>
+      <specular>0.1 0.1 0.1 1</specular>
+      <emissive>0 0 0 0</emissive>
+    </material>
+  </visual>
+</xacro:macro>
+<xacro:macro name="axle_color">
+  <visual>
+    <material>
+      <ambient>0.792156862745098 0.819607843137255 0.933333333333333 1</ambient>
+      <diffuse>0.792156862745098 0.819607843137255 0.933333333333333 1</diffuse>
+      <specular>0.1 0.1 0.1 1</specular>
+      <emissive>0 0 0 0</emissive>
+    </material>
+  </visual>
+</xacro:macro>
+<xacro:macro name="side_pane_color">
+  <visual>
+    <material>
+      <ambient>0.501960784313725 1 0.501960784313725 1</ambient>
+      <diffuse>0.501960784313725 1 0.501960784313725 1</diffuse>
+      <specular>0.1 0.1 0.1 1</specular>
+      <emissive>0 0 0 0</emissive>
+    </material>
+  </visual>
+</xacro:macro>
+<xacro:macro name="top_color">
+  <visual>
+    <material>
+      <ambient>0 0.752941176470588 0 1</ambient>
+      <diffuse>0 0.752941176470588 0 1</diffuse>
+      <specular>0.1 0.1 0.1 1</specular>
+      <emissive>0 0 0 0</emissive>
+    </material>
+  </visual>
+</xacro:macro>
+<xacro:macro name="wheel_color">
+  <visual>
+    <material>
+      <ambient>0 0 0 1</ambient>
+      <diffuse>0 0 0 1</diffuse>
+      <specular>0.1 0.1 0.1 1</specular>
+      <emissive>0 0 0 0</emissive>
+    </material>
+  </visual>
+</xacro:macro>
+<xacro:macro name="lidar_color">
+  <visual>
+    <material>
+      <ambient>0 0 0 1</ambient>
+      <diffuse>0 0 0 1</diffuse>
+      <specular>0.1 0.1 0.1 1</specular>
+      <emissive>0 0 0 0</emissive>
+    </material>
+  </visual>
+</xacro:macro>
   <link
     name="body">
     <inertial>
       <origin
-        xyz="-3.40969326113787E-05 -1.55139179626814E-05 0.984476420828284"
-        rpy="0 0 0" />
-      <mass
-        value="7062.99841256932" />
-      <inertia
-        ixx="2779.69153524293"
-        ixy="0.0130537985025844"
-        ixz="-0.074560285709414"
-        iyy="11898.0975209909"
-        iyz="-0.0273565484571444"
-        izz="12806.0341693142" />
+        xyz="-5.21780361655602E-05 -2.37407212439023E-05 0.604812969920948"
+        rpy="0 0 0" />
+      <mass
+        value="4615.47805567614" />
+      <inertia
+        ixx="1863.24455406167"
+        ixy="0.0132219930650718"
+        ixz="-0.0745602857100425"
+        iyy="8715.44296968045"
+        iyz="-0.0273565484550983"
+        izz="9003.50747380204" />
     </inertial>
     <visual>
@@ -31,5 +92,5 @@
         name="">
         <color
-          rgba="0.792156862745098 0.819607843137255 0.933333333333333 1" />
+          rgba="0.250980392156863 0.250980392156863 0.250980392156863 1" />
       </material>
     </visual>
@@ -106,14 +167,14 @@
     <inertial>
       <origin
-        xyz="-1.58019056769578 -1.04124193078514 0.309999999999997"
+        xyz="1.57025410376083 -1.04055974237639 0.309999999999996"
         rpy="0 0 0" />
       <mass
         value="220.204654088327" />
       <inertia
-        ixx="19.6593954325899"
-        ixy="-0.775721213261626"
-        ixz="-1.12534049438089E-15"
-        iyy="33.7627965853084"
-        iyz="5.12575321634251E-14"
+        ixx="19.7127728680101"
+        ixy="1.16262531983733"
+        ixz="5.70065896608079E-15"
+        iyy="33.7094191498882"
+        iyz="5.93281734338829E-14"
         izz="19.6168571900673" />
     </inertial>
@@ -153,5 +214,5 @@
       link="front_right_wheel" />
     <axis
-      xyz="0.08222 0.99661 0" />
+      xyz="0.0822198916962624 0.996614212927678 0" />
     <limit
       lower="0"
@@ -228,8 +289,8 @@
       <inertia
         ixx="25.1304300235974"
-        ixy="6.91590337281264"
-        ixz="2.62007454425615E-14"
+        ixy="6.91590337281265"
+        ixz="2.78109008982202E-14"
         iyy="28.2917619943008"
-        iyz="3.1857375012075E-14"
+        iyz="2.83392710451218E-14"
         izz="19.6168571900673" />
     </inertial>
@@ -269,5 +330,5 @@
       link="front_left_wheel" />
     <axis
-      xyz="-0.62337 -0.78192 0" />
+      xyz="-0.623373961813521 -0.781923847783731 0" />
     <limit
       lower="0"
@@ -341,11 +402,11 @@
         rpy="0 0 0" />
       <mass
-        value="220.204654088326" />
+        value="220.204654088327" />
       <inertia
         ixx="19.7817557340667"
         ixy="1.52068003676715"
-        ixz="-1.46712089567244E-16"
+        ixz="-1.41066843422813E-16"
         iyy="33.6404362838315"
-        iyz="5.3547004248261E-14"
+        iyz="5.35623170831363E-14"
         izz="19.6168571900673" />
     </inertial>
@@ -385,5 +446,5 @@
       link="back_left_wheel" />
     <axis
-      xyz="-0.10781 -0.99417 0" />
+      xyz="-0.107805398797207 -0.99417201529221 0" />
     <limit
       lower="0"
@@ -461,7 +522,7 @@
         ixx="19.6593954325899"
         ixy="-0.775721213261626"
-        ixz="-1.12757594335517E-15"
+        ixz="-1.12449279054662E-15"
         iyy="33.7627965853084"
-        iyz="5.12534151456868E-14"
+        iyz="5.12487286095604E-14"
         izz="19.6168571900673" />
     </inertial>
@@ -501,5 +562,5 @@
       link="back_right_wheel" />
     <axis
-      xyz="-0.054755 0.9985 0" />
+      xyz="-0.0547547589597665 0.998499832935018 0" />
     <limit
       lower="0"
@@ -518,8 +579,8 @@
       <inertia
         ixx="0.0642189157299355"
-        ixy="-0.000191353707477662"
-        ixz="0.00017449312202714"
+        ixy="-0.000191353707477661"
+        ixz="0.000174493122027139"
         iyy="0.0642189157299355"
-        iyz="-0.000174493122027057"
+        iyz="-0.000174493122027053"
         izz="0.0429541548113749" />
     </inertial>
@@ -571,8 +632,8 @@
       <inertia
         ixx="0.0642189157299355"
-        ixy="0.00019135370747766"
+        ixy="0.000191353707477661"
         ixz="0.000174493122027142"
         iyy="0.0642189157299355"
-        iyz="0.000174493122027216"
+        iyz="0.000174493122027214"
         izz="0.0429541548113749" />
     </inertial>
@@ -671,5 +732,5 @@
     <inertial>
       <origin
-        xyz="-2.10240622729716 -1.10240622729718 1.78815355406656"
+        xyz="-2.10240622729716 -1.10240622729717 1.78815355406656"
         rpy="0 0 0" />
       <mass
@@ -720,3 +781,322 @@
       xyz="0 0 0" />
   </joint>
+  <link
+    name="side_pane_1">
+    <inertial>
+      <origin
+        xyz="1.19387690613411E-15 0.939999999999996 1.22578533508363"
+        rpy="0 0 0" />
+      <mass
+        value="269.579902102743" />
+      <inertia
+        ixx="29.0495518679719"
+        ixy="-1.20383938267813E-16"
+        ixz="3.27421223583015E-14"
+        iyy="417.804106229136"
+        iyz="9.89684859766926E-14"
+        izz="389.401546126211" />
+    </inertial>
+    <visual>
+      <origin
+        xyz="0 0 0"
+        rpy="0 0 0" />
+      <geometry>
+        <mesh
+          filename="package://project_legion/meshes/side_pane_1.STL" />
+      </geometry>
+      <material
+        name="">
+        <color
+          rgba="0.792156862745098 0.819607843137255 0.933333333333333 1" />
+      </material>
+    </visual>
+    <collision>
+      <origin
+        xyz="0 0 0"
+        rpy="0 0 0" />
+      <geometry>
+        <mesh
+          filename="package://project_legion/meshes/side_pane_1.STL" />
+      </geometry>
+    </collision>
+  </link>
+  <joint
+    name="side_pane_1_joint"
+    type="fixed">
+    <origin
+      xyz="0 0 0"
+      rpy="0 0 0" />
+    <parent
+      link="body" />
+    <child
+      link="side_pane_1" />
+    <axis
+      xyz="0 0 0" />
+  </joint>
+  <link
+    name="side_pane_2">
+    <inertial>
+      <origin
+        xyz="7.36854275917892E-17 -0.940000000000004 1.22578533508363"
+        rpy="0 0 0" />
+      <mass
+        value="269.579902102743" />
+      <inertia
+        ixx="29.0495518679719"
+        ixy="-1.20383938267801E-16"
+        ixz="2.9415137108934E-14"
+        iyy="417.804106229136"
+        iyz="9.89935929190605E-14"
+        izz="389.401546126211" />
+    </inertial>
+    <visual>
+      <origin
+        xyz="0 0 0"
+        rpy="0 0 0" />
+      <geometry>
+        <mesh
+          filename="package://project_legion/meshes/side_pane_2.STL" />
+      </geometry>
+      <material
+        name="">
+        <color
+          rgba="0.792156862745098 0.819607843137255 0.933333333333333 1" />
+      </material>
+    </visual>
+    <collision>
+      <origin
+        xyz="0 0 0"
+        rpy="0 0 0" />
+      <geometry>
+        <mesh
+          filename="package://project_legion/meshes/side_pane_2.STL" />
+      </geometry>
+    </collision>
+  </link>
+  <joint
+    name="side_pane_2_joint"
+    type="fixed">
+    <origin
+      xyz="0 0 0"
+      rpy="0 0 0" />
+    <parent
+      link="body" />
+    <child
+      link="side_pane_2" />
+    <axis
+      xyz="0 0 0" />
+  </joint>
+  <link
+    name="side_pane_3">
+    <inertial>
+      <origin
+        xyz="-1.94 -4.0299328481463E-15 1.16174583422535"
+        rpy="0 0 0" />
+      <mass
+        value="238.283902102743" />
+      <inertia
+        ixx="91.2445420486072"
+        ixy="-2.58236719045494E-16"
+        ixz="1.67397202198221E-16"
+        iyy="30.1909069158719"
+        iyz="-1.1589443866755E-13"
+        izz="61.6255164977819" />
+    </inertial>
+    <visual>
+      <origin
+        xyz="0 0 0"
+        rpy="0 0 0" />
+      <geometry>
+        <mesh
+          filename="package://project_legion/meshes/side_pane_3.STL" />
+      </geometry>
+      <material
+        name="">
+        <color
+          rgba="0.792156862745098 0.819607843137255 0.933333333333333 1" />
+      </material>
+    </visual>
+    <collision>
+      <origin
+        xyz="0 0 0"
+        rpy="0 0 0" />
+      <geometry>
+        <mesh
+          filename="package://project_legion/meshes/side_pane_3.STL" />
+      </geometry>
+    </collision>
+  </link>
+  <joint
+    name="side_pane_3_joint"
+    type="fixed">
+    <origin
+      xyz="0 0 0"
+      rpy="0 0 0" />
+    <parent
+      link="body" />
+    <child
+      link="side_pane_3" />
+    <axis
+      xyz="0 0 0" />
+  </joint>
+  <link
+    name="side_pane_4">
+    <inertial>
+      <origin
+        xyz="8.11876186905901E-17 -0.16174583422535 -0.0599999999999998"
+        rpy="0 0 0" />
+      <mass
+        value="238.283902102743" />
+      <inertia
+        ixx="30.1909069158719"
+        ixy="-1.35061898246685E-14"
+        ixz="3.03407211392029E-16"
+        iyy="61.6255164977819"
+        iyz="4.1134269100746E-16"
+        izz="91.2445420486072" />
+    </inertial>
+    <visual>
+      <origin
+        xyz="0 0 0"
+        rpy="0 0 0" />
+      <geometry>
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
Commit message: Task 1.3.3.0: Test Controllers

File: urdf/robotaxi.urdf.xacro (robot description, xacro)
@@ -1100,3 +1100,27 @@
     <xacro:top_color />
   </gazebo>
+  <!-- Adding Controllers -->
+  <ros2_control name="GazeboSystem" type="system">
+  <hardware>
+    <plugin>gazebo_ros2_control/GazeboSystem</plugin>
+  </hardware>
+  <joint name="back_right_wheel_joint">
+    <command_interface name="position">
+        <param name="min">-0.05</param>
+        <param name="max">0.0</param>
+    </command_interface>
+    <state_interface name="position"/>
+    <state_interface name="velocity"/>
+    <state_interface name="effort"/>
+  </joint>
+  </ros2_control>
+  <gazebo>
+      <plugin filename="libgazebo_ros2_control.so" name="gazebo_ros2_control">
+        <ros>
+          <namespace>/robotaxi</namespace>
+        </ros>
+        <robot_param_node>/robotaxi_robot_state_publisher</robot_param_node>
+        <parameters>$(find project_legion)/config/control.yaml</parameters>
+      </plugin>
+  </gazebo>
 </robot>

Commit message: Task 1.3.3:  Added Controllers to Model

File: urdf/robotaxi.urdf.xacro (robot description, xacro)
@@ -205,5 +205,5 @@
   <joint
     name="front_right_wheel_joint"
-    type="revolute">
+    type="continuous">
     <origin
       xyz="0 0 0"
@@ -321,5 +321,5 @@
   <joint
     name="front_left_wheel_joint"
-    type="revolute">
+    type="continuous">
     <origin
       xyz="0 0 0"
@@ -437,5 +437,5 @@
   <joint
     name="back_left_wheel_joint"
-    type="revolute">
+    type="continuous">
     <origin
       xyz="0 0 0"
@@ -553,5 +553,5 @@
   <joint
     name="back_right_wheel_joint"
-    type="revolute">
+    type="continuous">
     <origin
       xyz="0 0 0"
@@ -1106,19 +1106,38 @@
   </hardware>
   <joint name="back_right_wheel_joint">
-    <command_interface name="position">
-        <param name="min">-0.05</param>
-        <param name="max">0.0</param>
+    <command_interface name="velocity">
+        <param name="min">-1000.0</param>
+        <param name="max">1000.0</param>
     </command_interface>
     <state_interface name="position"/>
     <state_interface name="velocity"/>
-    <state_interface name="effort"/>
+  </joint>
+  <joint name="front_right_wheel_joint">
+    <command_interface name="velocity">
+        <param name="min">-1000.0</param>
+        <param name="max">1000.0</param>
+    </command_interface>
+    <state_interface name="position"/>
+    <state_interface name="velocity"/>
+  </joint>
+  <joint name="back_left_wheel_joint">
+    <command_interface name="velocity">
+        <param name="min">-1000.0</param>
+        <param name="max">1000.0</param>
+    </command_interface>
+    <state_interface name="position"/>
+    <state_interface name="velocity"/>
+  </joint>
+  <joint name="front_left_wheel_joint">
+    <command_interface name="velocity">
+        <param name="min">-1000.0</param>
+        <param name="max">1000.0</param>
+    </command_interface>
+    <state_interface name="position"/>
+    <state_interface name="velocity"/>
   </joint>
   </ros2_control>
   <gazebo>
       <plugin filename="libgazebo_ros2_control.so" name="gazebo_ros2_control">
-        <ros>
-          <namespace>/robotaxi</namespace>
-        </ros>
-        <robot_param_node>/robotaxi_robot_state_publisher</robot_param_node>
         <parameters>$(find project_legion)/config/control.yaml</parameters>
       </plugin>
