Commit message: Task 1.3.4: Successfully Added  Controllers

File: urdf/robotaxi.urdf.xacro (robot description, xacro)
@@ -1,73 +1,73 @@
-<?xml version="1.0"?>
+<?xml version="1.0" ?>
 <!-- This URDF was automatically created by SolidWorks to URDF Exporter! Originally created by Stephen Brawner (brawner@gmail.com)
      Commit Version: 1.6.0-4-g7f85cfe  Build Version: 1.6.7995.38578
      For more information, please see http://wiki.ros.org/sw_urdf_exporter -->
 <robot
-  name="robotaxi">
+  name="robotaxi" xmlns:xacro="http://ros.org/wiki/xacro">
   <xacro:macro name="body_color">
-  <visual>
-    <material>
-      <ambient>0.250980392156863 0.250980392156863 0.250980392156863 1</ambient>
-      <diffuse>0.250980392156863 0.250980392156863 0.250980392156863 1</diffuse>
-      <specular>0.1 0.1 0.1 1</specular>
-      <emissive>0 0 0 0</emissive>
-    </material>
-  </visual>
-</xacro:macro>
-<xacro:macro name="axle_color">
-  <visual>
-    <material>
-      <ambient>0.792156862745098 0.819607843137255 0.933333333333333 1</ambient>
-      <diffuse>0.792156862745098 0.819607843137255 0.933333333333333 1</diffuse>
-      <specular>0.1 0.1 0.1 1</specular>
-      <emissive>0 0 0 0</emissive>
-    </material>
-  </visual>
-</xacro:macro>
-<xacro:macro name="side_pane_color">
-  <visual>
-    <material>
-      <ambient>0.501960784313725 1 0.501960784313725 1</ambient>
-      <diffuse>0.501960784313725 1 0.501960784313725 1</diffuse>
-      <specular>0.1 0.1 0.1 1</specular>
-      <emissive>0 0 0 0</emissive>
-    </material>
-  </visual>
-</xacro:macro>
-<xacro:macro name="top_color">
-  <visual>
-    <material>
-      <ambient>0 0.752941176470588 0 1</ambient>
-      <diffuse>0 0.752941176470588 0 1</diffuse>
-      <specular>0.1 0.1 0.1 1</specular>
-      <emissive>0 0 0 0</emissive>
-    </material>
-  </visual>
-</xacro:macro>
-<xacro:macro name="wheel_color">
-  <visual>
-    <material>
-      <ambient>0 0 0 1</ambient>
-      <diffuse>0 0 0 1</diffuse>
-      <specular>0.1 0.1 0.1 1</specular>
-      <emissive>0 0 0 0</emissive>
-    </material>
-  </visual>
-</xacro:macro>
-<xacro:macro name="lidar_color">
-  <visual>
-    <material>
-      <ambient>0 0 0 1</ambient>
-      <diffuse>0 0 0 1</diffuse>
-      <specular>0.1 0.1 0.1 1</specular>
-      <emissive>0 0 0 0</emissive>
-    </material>
-  </visual>
-</xacro:macro>
-  <link
-    name="body">
-    <inertial>
-      <origin
-        xyz="-5.21780361656553E-05 -2.37407212439034E-05 0.604812969920948"
+    <visual>
+      <material>
+        <ambient>0.250980392156863 0.250980392156863 0.250980392156863 1</ambient>
+        <diffuse>0.250980392156863 0.250980392156863 0.250980392156863 1</diffuse>
+        <specular>0.1 0.1 0.1 1</specular>
+        <emissive>0 0 0 0</emissive>
+      </material>
+    </visual>
+  </xacro:macro>
+  <xacro:macro name="axle_color">
+    <visual>
+      <material>
+        <ambient>0.792156862745098 0.819607843137255 0.933333333333333 1</ambient>
+        <diffuse>0.792156862745098 0.819607843137255 0.933333333333333 1</diffuse>
+        <specular>0.1 0.1 0.1 1</specular>
+        <emissive>0 0 0 0</emissive>
+      </material>
+    </visual>
+  </xacro:macro>
+  <xacro:macro name="side_pane_color">
+    <visual>
+      <material>
+        <ambient>0.501960784313725 1 0.501960784313725 1</ambient>
+        <diffuse>0.501960784313725 1 0.501960784313725 1</diffuse>
+        <specular>0.1 0.1 0.1 1</specular>
+        <emissive>0 0 0 0</emissive>
+      </material>
+    </visual>
+  </xacro:macro>
+  <xacro:macro name="top_color">
+    <visual>
+      <material>
+        <ambient>0 0.752941176470588 0 1</ambient>
+        <diffuse>0 0.752941176470588 0 1</diffuse>
+        <specular>0.1 0.1 0.1 1</specular>
+        <emissive>0 0 0 0</emissive>
+      </material>
+    </visual>
+  </xacro:macro>
+  <xacro:macro name="wheel_color">
+    <visual>
+      <material>
+        <ambient>0 0 0 1</ambient>
+        <diffuse>0 0 0 1</diffuse>
+        <specular>0.1 0.1 0.1 1</specular>
+        <emissive>0 0 0 0</emissive>
+      </material>
+    </visual>
+  </xacro:macro>
+  <xacro:macro name="lidar_color">
+    <visual>
+      <material>
+        <ambient>0 0 0 1</ambient>
+        <diffuse>0 0 0 1</diffuse>
+        <specular>0.1 0.1 0.1 1</specular>
+        <emissive>0 0 0 0</emissive>
+      </material>
+    </visual>
+  </xacro:macro>
+  <link
+    name="base_link">
+    <inertial>
+      <origin
+        xyz="-5.2178036165576E-05 -2.37407212439011E-05 0.604812969920948"
         rpy="0 0 0" />
       <mass
@@ -75,8 +75,8 @@
       <inertia
         ixx="1863.24455406167"
-        ixy="0.0132219930650691"
-        ixz="-0.0745602857101254"
+        ixy="0.0132219930650514"
+        ixz="-0.0745602857101196"
         iyy="8715.44296968045"
-        iyz="-0.0273565484551131"
+        iyz="-0.0273565484551048"
         izz="9003.50747380203" />
     </inertial>
@@ -87,5 +87,5 @@
       <geometry>
         <mesh
-          filename="package://project_legion/meshes/body.STL" />
+          filename="package://project_legion/meshes/base_link.STL" />
       </geometry>
       <material
@@ -101,5 +101,5 @@
       <geometry>
         <mesh
-          filename="package://project_legion/meshes/body.STL" />
+          filename="package://project_legion/meshes/base_link.STL" />
       </geometry>
     </collision>
@@ -109,15 +109,15 @@
     <inertial>
       <origin
-        xyz="-0.00745692269118803 -0.090387884139878 0.106936663484027"
-        rpy="0 0 0" />
-      <mass
-        value="4.73802510796172" />
-      <inertia
-        ixx="0.0990829916203824"
-        ixy="-0.00564103885906436"
-        ixz="0.000108229508691783"
-        iyy="0.0311714791660352"
-        iyz="0.00131190404983014"
-        izz="0.106577267989412" />
+        xyz="7.22269732911229E-09 -0.0906949566483326 0.106936664568276"
+        rpy="0 0 0" />
+      <mass
+        value="4.73802510742154" />
+      <inertia
+        ixx="0.0995483725414788"
+        ixy="1.31296102047959E-09"
+        ixz="-1.57301902386985E-09"
+        iyy="0.0307060985233193"
+        iyz="0.0013163608882011"
+        izz="0.106577268300346" />
     </inertial>
     <visual>
@@ -149,8 +149,8 @@
     type="revolute">
     <origin
-      xyz="1.6 -0.680000000000001 0.199999999999998"
-      rpy="0 0 0" />
-    <parent
-      link="body" />
+      xyz="1.6 -0.68 0.2"
+      rpy="0 0 0" />
+    <parent
+      link="base_link" />
     <child
       link="front_right_axel" />
@@ -158,8 +158,8 @@
       xyz="0 0 1" />
     <limit
-      lower="0"
-      upper="0"
-      effort="0"
-      velocity="0" />
+      lower="-3.14"
+      upper="3.14"
+      effort="100"
+      velocity="1000" />
   </joint>
   <link
@@ -167,14 +167,14 @@
     <inertial>
       <origin
-        xyz="-6.45153368084017E-05 -0.000782011509483205 -1.11022302462516E-16"
+        xyz="0 -0.000784668229028895 -1.11022302462516E-16"
         rpy="0 0 0" />
       <mass
         value="220.204654088327" />
       <inertia
-        ixx="19.7127728680101"
-        ixy="1.16262531983733"
-        ixz="5.60424286950757E-15"
-        iyy="33.7094191498882"
-        iyz="5.89373897821999E-14"
+        ixx="19.6168571900673"
+        ixy="1.10879109651903E-15"
+        ixz="5.72594272343911E-16"
+        iyy="33.8053348278309"
+        iyz="4.98336858770083E-14"
         izz="19.6168571900673" />
     </inertial>
@@ -205,7 +205,7 @@
   <joint
     name="front_right_wheel_joint"
-    type="revolute">
-    <origin
-      xyz="-0.0296813809023602 -0.359777730866907 0.109999999999998"
+    type="continuous">
+    <origin
+      xyz="0 -0.361 0.11"
       rpy="0 0 0" />
     <parent
@@ -214,10 +214,5 @@
       link="front_right_wheel" />
     <axis
-      xyz="0.0822198916962624 0.996614212927678 0" />
-    <limit
-      lower="0"
-      upper="0"
-      effort="0"
-      velocity="0" />
+      xyz="0 1 0" />
   </joint>
   <link
@@ -225,15 +220,15 @@
     <inertial>
       <origin
-        xyz="0.0565368692558958 0.0709165541990985 0.106936664135948"
-        rpy="0 0 0" />
-      <mass
-        value="4.73802513910441" />
-      <inertia
-        ixx="0.0727966036899852"
-        ixy="-0.033555856058096"
-        ixz="-0.0008205838617529"
-        iyy="0.0574578673139121"
-        iyz="-0.00102929493752076"
-        izz="0.106577268204647" />
+        xyz="-7.22269799524611E-09 0.0906949566483317 0.106936664568277"
+        rpy="0 0 0" />
+      <mass
+        value="4.73802510742154" />
+      <inertia
+        ixx="0.0995483725414789"
+        ixy="1.31296104323952E-09"
+        ixz="1.57301903314861E-09"
+        iyy="0.0307060985233193"
+        iyz="-0.00131636088820162"
+        izz="0.106577268300346" />
     </inertial>
     <visual>
@@ -265,8 +260,8 @@
     type="revolute">
     <origin
-      xyz="1.6 0.68 0.200000000000002"
-      rpy="0 0 0" />
-    <parent
-      link="body" />
+      xyz="1.6 0.68 0.2"
+      rpy="0 0 0" />
+    <parent
+      link="base_link" />
     <child
       link="front_left_axel" />
@@ -274,8 +269,8 @@
       xyz="0 0 1" />
     <limit
-      lower="0"
-      upper="0"
-      effort="0"
-      velocity="0" />
+      lower="-3.14"
+      upper="3.14"
+      effort="100"
+      velocity="1000" />
   </joint>
   <link
@@ -283,14 +278,125 @@
     <inertial>
       <origin
-        xyz="0.000489141742639143 0.000613550800876106 -5.55111512312578E-17"
+        xyz="2.22044604925031E-16 0.000784668229028895 0"
+        rpy="0 0 0" />
+      <mass
+        value="220.204654088326" />
+      <inertia
+        ixx="19.6168571900673"
+        ixy="-2.0242871863207E-15"
+        ixz="1.40172771935682E-15"
+        iyy="33.8053348278309"
+        iyz="4.94762339235896E-14"
+        izz="19.6168571900673" />
+    </inertial>
+    <visual>
+      <origin
+        xyz="0 0 0"
+        rpy="0 0 0" />
+      <geometry>
+        <mesh
+          filename="package://project_legion/meshes/front_left_wheel.STL" />
+      </geometry>
+      <material
+        name="">
+        <color
+          rgba="0.792156862745098 0.819607843137255 0.933333333333333 1" />
+      </material>
+    </visual>
+    <collision>
+      <origin
+        xyz="0 0 0"
+        rpy="0 0 0" />
+      <geometry>
+        <mesh
+          filename="package://project_legion/meshes/front_left_wheel.STL" />
+      </geometry>
+    </collision>
+  </link>
+  <joint
+    name="front_left_wheel_joint"
+    type="continuous">
+    <origin
+      xyz="0 0.361 0.110000000000001"
+      rpy="0 0 0" />
+    <parent
+      link="front_left_axel" />
+    <child
+      link="front_left_wheel" />
+    <axis
+      xyz="0 -1 0" />
+  </joint>
+  <link
+    name="back_right_axel">
+    <inertial>
+      <origin
+        xyz="7.22269732911229E-09 -0.0906949566483326 0.106936664568276"
+        rpy="0 0 0" />
+      <mass
+        value="4.73802510742154" />
+      <inertia
+        ixx="0.0995483725414788"
+        ixy="1.31296104260797E-09"
+        ixz="-1.57301902354649E-09"
+        iyy="0.0307060985233193"
+        iyz="0.00131636088820109"
+        izz="0.106577268300346" />
+    </inertial>
+    <visual>
+      <origin
+        xyz="0 0 0"
+        rpy="0 0 0" />
+      <geometry>
+        <mesh
+          filename="package://project_legion/meshes/back_right_axel.STL" />
+      </geometry>
+      <material
+        name="">
+        <color
+          rgba="0.792156862745098 0.819607843137255 0.933333333333333 1" />
+      </material>
+    </visual>
+    <collision>
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
Commit message: RVIZ Changes

File: urdf/robotaxi.urdf.xacro (robot description, xacro)
@@ -65,4 +65,6 @@
     </visual>
   </xacro:macro>
+  <link name="dummy_link">
+    </link>
   <link
     name="base_link">
@@ -90,5 +92,5 @@
       </geometry>
       <material
-        name="">
+        name="body_mat">
         <color
           rgba="0.250980392156863 0.250980392156863 0.250980392156863 1" />
@@ -105,4 +107,8 @@
     </collision>
   </link>
+  <joint name="dummy_joint" type="fixed">
+        <parent link="dummy_link"/>
+        <child link="base_link"/>
+  </joint>
   <link
     name="front_right_axel">
@@ -130,5 +136,5 @@
       </geometry>
       <material
-        name="">
+        name="axel_mat">
         <color
           rgba="0.792156862745098 0.819607843137255 0.933333333333333 1" />
@@ -188,5 +194,5 @@
       </geometry>
       <material
-        name="">
+        name="wheel_mat">
         <color
           rgba="0.792156862745098 0.819607843137255 0.933333333333333 1" />
@@ -241,5 +247,5 @@
       </geometry>
       <material
-        name="">
+        name="axel_mat">
         <color
           rgba="0.792156862745098 0.819607843137255 0.933333333333333 1" />
@@ -299,5 +305,5 @@
       </geometry>
       <material
-        name="">
+        name="wheel_mat">
         <color
           rgba="0.792156862745098 0.819607843137255 0.933333333333333 1" />
@@ -352,5 +358,5 @@
       </geometry>
       <material
-        name="">
+        name="axel_mat">
         <color
           rgba="0.792156862745098 0.819607843137255 0.933333333333333 1" />
@@ -410,5 +416,5 @@
       </geometry>
       <material
-        name="">
+        name="wheel_mat">
         <color
           rgba="0.792156862745098 0.819607843137255 0.933333333333333 1" />
@@ -463,5 +469,5 @@
       </geometry>
       <material
-        name="">
+        name="axel_mat">
         <color
           rgba="0.792156862745098 0.819607843137255 0.933333333333333 1" />
@@ -521,5 +527,5 @@
       </geometry>
       <material
-        name="">
+        name="wheel_mat">
         <color
           rgba="0.792156862745098 0.819607843137255 0.933333333333333 1" />
@@ -574,5 +580,5 @@
       </geometry>
       <material
-        name="">
+        name="side_mat">
         <color
           rgba="0.792156862745098 0.819607843137255 0.933333333333333 1" />
@@ -627,5 +633,5 @@
       </geometry>
       <material
-        name="">
+        name="side_mat_1">
         <color
           rgba="0.792156862745098 0.819607843137255 0.933333333333333 1" />
@@ -680,5 +686,5 @@
       </geometry>
       <material
-        name="">
+        name="side_mat_2">
         <color
           rgba="0.792156862745098 0.819607843137255 0.933333333333333 1" />
@@ -733,5 +739,5 @@
       </geometry>
       <material
-        name="">
+        name="side_mat_3">
         <color
           rgba="0.792156862745098 0.819607843137255 0.933333333333333 1" />
@@ -786,5 +792,5 @@
       </geometry>
       <material
-        name="">
+        name="top_mat">
         <color
           rgba="0.792156862745098 0.819607843137255 0.933333333333333 1" />
@@ -839,5 +845,5 @@
       </geometry>
       <material
-        name="">
+        name="lidar_mat">
         <color
           rgba="0.792156862745098 0.819607843137255 0.933333333333333 1" />
@@ -892,5 +898,5 @@
       </geometry>
       <material
-        name="">
+        name="lidar_mat">
         <color
           rgba="0.792156862745098 0.819607843137255 0.933333333333333 1" />
@@ -945,5 +951,5 @@
       </geometry>
       <material
-        name="">
+        name="lidar_mat">
         <color
           rgba="0.792156862745098 0.819607843137255 0.933333333333333 1" />
@@ -998,5 +1004,5 @@
       </geometry>
       <material
-        name="">
+        name="lidar_mat">
         <color
           rgba="0.792156862745098 0.819607843137255 0.933333333333333 1" />
@@ -1155,3 +1161,143 @@
       </plugin>
   </gazebo>
+  <gazebo reference="front_left_lidar">
+  <sensor name="lidar" type="ray">
+    <pose>0.215 0 0.215 0 0 0</pose>
+    <always_on>true</always_on>
+    <visualize>false</visualize>
+    <update_rate>5</update_rate>
+    <ray>
+      <scan>
+        <horizontal>
+          <samples>360</samples>
+          <resolution>1.00000</resolution>
+          <min_angle>0.000000</min_angle>
+          <max_angle>6.280000</max_angle>
+        </horizontal>
+      </scan>
+      <range>
+        <min>0.120000</min>
+        <max>3.5</max>
+        <resolution>0.015000</resolution>
+      </range>
+      <noise>
+        <type>gaussian</type>
+        <mean>0.0</mean>
+        <stddev>0.01</stddev>
+      </noise>
+    </ray>
+    <plugin name="scan_1" filename="libgazebo_ros_ray_sensor.so">
+      <ros>
+        <remapping>~/out:=scan_1</remapping>
+      </ros>
+      <output_type>sensor_msgs/LaserScan</output_type>
+      <frame_name>front_left_lidar</frame_name>
+    </plugin>
+  </sensor>
+  </gazebo>
+  <gazebo reference="back_right_lidar">
+  <sensor name="lidar" type="ray">
+    <pose>0.215 0 0.215 0 0 0</pose>
+    <always_on>true</always_on>
+    <visualize>false</visualize>
+    <update_rate>5</update_rate>
+    <ray>
+      <scan>
+        <horizontal>
+          <samples>360</samples>
+          <resolution>1.00000</resolution>
+          <min_angle>0.000000</min_angle>
+          <max_angle>6.280000</max_angle>
+        </horizontal>
+      </scan>
+      <range>
+        <min>0.120000</min>
+        <max>3.5</max>
+        <resolution>0.015000</resolution>
+      </range>
+      <noise>
+        <type>gaussian</type>
+        <mean>0.0</mean>
+        <stddev>0.01</stddev>
+      </noise>
+    </ray>
+    <plugin name="scan_2" filename="libgazebo_ros_ray_sensor.so">
+      <ros>
+        <remapping>~/out:=scan_2</remapping>
+      </ros>
+      <output_type>sensor_msgs/LaserScan</output_type>
+      <frame_name>back_right_lidar</frame_name>
+    </plugin>
+  </sensor>
+  </gazebo>
+  <gazebo reference="back_left_lidar">
+  <sensor name="lidar" type="ray">
+    <pose>0.215 0 0.215 0 0 0</pose>
+    <always_on>true</always_on>
+    <visualize>false</visualize>
+    <update_rate>5</update_rate>
+    <ray>
+      <scan>
+        <horizontal>
+          <samples>360</samples>
+          <resolution>1.00000</resolution>
+          <min_angle>0.000000</min_angle>
+          <max_angle>6.280000</max_angle>
+        </horizontal>
+      </scan>
+      <range>
+        <min>0.120000</min>
+        <max>3.5</max>
+        <resolution>0.015000</resolution>
+      </range>
+      <noise>
+        <type>gaussian</type>
+        <mean>0.0</mean>
+        <stddev>0.01</stddev>
+      </noise>
+    </ray>
+    <plugin name="scan_3" filename="libgazebo_ros_ray_sensor.so">
+      <ros>
+        <remapping>~/out:=scan_3</remapping>
+      </ros>
+      <output_type>sensor_msgs/LaserScan</output_type>
+      <frame_name>back_left_lidar</frame_name>
+    </plugin>
+  </sensor>
+  </gazebo>
+  <gazebo reference="front_right_lidar">
+  <sensor name="lidar" type="ray">
+    <pose>0.215 0 0.215 0 0 0</pose>
+    <always_on>true</always_on>
+    <visualize>false</visualize>
+    <update_rate>5</update_rate>
+    <ray>
+      <scan>
+        <horizontal>
+          <samples>360</samples>
+          <resolution>1.00000</resolution>
+          <min_angle>0.000000</min_angle>
+          <max_angle>6.280000</max_angle>
+        </horizontal>
+      </scan>
+      <range>
+        <min>0.120000</min>
+        <max>3.5</max>
+        <resolution>0.015000</resolution>
+      </range>
+      <noise>
+        <type>gaussian</type>
+        <mean>0.0</mean>
+        <stddev>0.01</stddev>
+      </noise>
+    </ray>
+    <plugin name="scan_4" filename="libgazebo_ros_ray_sensor.so">
+      <ros>
+        <remapping>~/out:=scan_4</remapping>
+      </ros>
+      <output_type>sensor_msgs/LaserScan</output_type>
+      <frame_name>front_right_lidar</frame_name>
+    </plugin>
+  </sensor>
+  </gazebo>
 </robot>

Commit message: Clean Up and Add Ons

File: urdf/robotaxi.urdf.xacro (robot description, xacro)
@@ -108,4 +108,5 @@
   </link>
   <joint name="dummy_joint" type="fixed">
+        <origin rpy="0 0 0" xyz="0 0 0" />
         <parent link="dummy_link"/>
         <child link="base_link"/>
